File: Controller/ESP32-S3_flipdot/ESP32-S3_flipdot.kicad_sch (KiCad schematic)
At the start: 6 parts, among them J1 Power in

Commit message: Before new dc-dc
Other:
- moved on the sheet: J1
Changed lines of the file:
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@@
     (stroke (width 0) (type default))
   )
-  (wire (pts (xy 67.691 160.02) (xy 67.691 163.068))
-    (stroke (width 0) (type default))
-  )
-  (wire (pts (xy 63.119 163.068) (xy 67.691 163.068))
-    (stroke (width 0) (type default))
-  )
-  (wire (pts (xy 63.119 165.608) (xy 67.691 165.608))
+  (wire (pts (xy 63.5 162.56) (xy 67.691 162.56))
     (stroke (width 0) (type default))
   )
@@
     (stroke (width 0) (type default))
   )
-  (wire (pts (xy 67.691 165.608) (xy 67.691 168.783))
-    (stroke (width 0) (type default))
-  )
-  (wire (pts (xy 71.882 160.02) (xy 67.691 160.02))
+  (wire (pts (xy 67.691 162.56) (xy 67.691 168.783))
+    (stroke (width 0) (type default))
+  )
+  (wire (pts (xy 63.5 160.02) (xy 71.882 160.02))
     (stroke (width 0) (type default))
   )
@@
     )
   )
-  (symbol (lib_id "Connector:Screw_Terminal_01x02") (at 58.039 163.068 0) (mirror y) (unit 1)
+  (symbol (lib_id "Connector:Screw_Terminal_01x02") (at 58.42 160.02 0) (mirror y) (unit 1)
     (in_bom yes) (on_board yes) (dnp no)
-    (property "Reference" "J1" (at 56.007 163.1259 0)
-      (effects (font (size 1.27 1.27)) (justify left))
-    )
-    (property "Value" "Power in" (at 56.007 165.5501 0)
-      (effects (font (size 1.27 1.27)) (justify left))
-    )
-    (property "Footprint" "TerminalBlock_Phoenix:TerminalBlock_Phoenix_MKDS-3-2-5.08_1x02_P5.08mm_Horizontal" (at 58.039 163.068 0)
-      (effects (font (size 1.27 1.27)) hide)
-    )
-    (property "Datasheet" "~" (at 58.039 163.068 0)
-      (effects (font (size 1.27 1.27)) hide)
-    )
-    (property "LCSC" "C5157144" (at 58.039 163.068 0)
-      (effects (font (size 1.27 1.27)) hide)
-    )
+    (property "Reference" "J1" (at 56.388 160.0779 0)
+      (effects (font (size 1.27 1.27)) (justify left))
+    )
+    (property "Value" "Power in" (at 56.388 162.5021 0)
+      (effects (font (size 1.27 1.27)) (justify left))
+    )
+    (property "Footprint" "TerminalBlock_Phoenix:TerminalBlock_Phoenix_MKDS-3-2-5.08_1x02_P5.08mm_Horizontal" (at 58.42 160.02 0)
+      (effects (font (size 1.27 1.27)) hide)
+    )
+    (property "Datasheet" "~" (at 58.42 160.02 0)
+      (effects (font (size 1.27 1.27)) hide)
+    )
+    (property "LCSC" "C5157144" (at 58.42 160.02 0)
+      (effects (font (size 1.27 1.27)) hide)
+    )

Commit message: WIP on PCB
Connections:
- net +5V: now also J1.2 (Pin_2); no longer J1.1 (Pin_1)
- net GND: now also J1.1 (Pin_1); no longer J1.2 (Pin_2)
Other:
- moved on the sheet: J1
Changed lines of the file:
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@@
     )
   )
-  (symbol (lib_id "Connector:Screw_Terminal_01x02") (at 58.42 160.02 0) (mirror y) (unit 1)
+  (symbol (lib_id "Connector:Screw_Terminal_01x02") (at 58.42 162.56 180) (unit 1)
     (in_bom yes) (on_board yes) (dnp no)
-    (property "Reference" "J1" (at 56.388 160.0779 0)
+    (property "Reference" "J1" (at 56.388 162.5021 0)
       (effects (font (size 1.27 1.27)) (justify left))
     )
-    (property "Value" "Power in" (at 56.388 162.5021 0)
+    (property "Value" "Power in" (at 56.388 160.0779 0)
       (effects (font (size 1.27 1.27)) (justify left))
     )
-    (property "Footprint" "TerminalBlock_Phoenix:TerminalBlock_Phoenix_MKDS-3-2-5.08_1x02_P5.08mm_Horizontal" (at 58.42 160.02 0)
+    (property "Footprint" "TerminalBlock_Phoenix:TerminalBlock_Phoenix_MKDS-3-2-5.08_1x02_P5.08mm_Horizontal" (at 58.42 162.56 0)
       (effects (font (size 1.27 1.27)) hide)
     )
-    (property "Datasheet" "~" (at 58.42 160.02 0)
+    (property "Datasheet" "~" (at 58.42 162.56 0)
       (effects (font (size 1.27 1.27)) hide)
     )
-    (property "LCSC" "C5157144" (at 58.42 160.02 0)
+    (property "LCSC" "C5157144" (at 58.42 162.56 0)
       (effects (font (size 1.27 1.27)) hide)
     )

Commit message: PCB in production!
Parts:
- H1, H2, H3, H4: now left out of the parts list
- J1: LCSC C5157144 -> C709041
Changed lines of the file:
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@@
   )
   (symbol (lib_id "Mechanical:MountingHole_Pad") (at 105.791 172.593 0) (unit 1)
-    (in_bom yes) (on_board yes) (dnp no) (fields_autoplaced)
+    (in_bom no) (on_board yes) (dnp no) (fields_autoplaced)
     (property "Reference" "H4" (at 108.331 170.1109 0)
       (effects (font (size 1.27 1.27)) (justify left))
@@
   )
   (symbol (lib_id "Mechanical:MountingHole_Pad") (at 129.032 173.228 0) (unit 1)
-    (in_bom yes) (on_board yes) (dnp no) (fields_autoplaced)
+    (in_bom no) (on_board yes) (dnp no) (fields_autoplaced)
     (property "Reference" "H2" (at 131.572 170.7459 0)
       (effects (font (size 1.27 1.27)) (justify left))
@@
   )
   (symbol (lib_id "Mechanical:MountingHole_Pad") (at 129.032 160.401 0) (unit 1)
-    (in_bom yes) (on_board yes) (dnp no) (fields_autoplaced)
+    (in_bom no) (on_board yes) (dnp no) (fields_autoplaced)
     (property "Reference" "H1" (at 131.572 157.9189 0)
       (effects (font (size 1.27 1.27)) (justify left))
@@
       (effects (font (size 1.27 1.27)) hide)
     )
-    (property "LCSC" "C5157144" (at 58.42 162.56 0)
+    (property "LCSC" "C709041" (at 58.42 162.56 0)
       (effects (font (size 1.27 1.27)) hide)
     )
@@
   )
   (symbol (lib_id "Mechanical:MountingHole_Pad") (at 105.537 159.766 0) (unit 1)
-    (in_bom yes) (on_board yes) (dnp no) (fields_autoplaced)
+    (in_bom no) (on_board yes) (dnp no) (fields_autoplaced)
     (property "Reference" "H3" (at 108.077 157.2839 0)
       (effects (font (size 1.27 1.27)) (justify left))
