File: Controller/ESP32-S3_flipdot/dc-dc.kicad_sch (KiCad schematic)
At the start: 31 parts, among them J3 BackLight, J5 BL_CMD, J6 BL_PWR, J7 COIL_PWR, Q3 2N3904, Q4 2N3904, Q5 ZXMP4A16G, Q6 ZXMP4A16G, U7 MT3608, U8 MT3608

Commit message: Before new dc-dc
Other:
- moved on the sheet: J7
Changed lines of the file:
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@@
   (junction (at 98.679 144.018) (diameter 0) (color 0 0 0 0)
   )
+  (junction (at 204.343 121.158) (diameter 0) (color 0 0 0 0)
+  )
   (junction (at 217.678 43.815) (diameter 0) (color 0 0 0 0)
   )
@@
     (stroke (width 0) (type default))
   )
-  (wire (pts (xy 204.343 121.031) (xy 204.343 128.651))
-    (stroke (width 0) (type default))
-  )
   (wire (pts (xy 118.999 109.347) (xy 103.759 109.347))
     (stroke (width 0) (type default))
@@
     (stroke (width 0) (type default))
   )
+  (wire (pts (xy 204.343 121.158) (xy 204.343 128.651))
+    (stroke (width 0) (type default))
+  )
   (wire (pts (xy 228.473 54.483) (xy 227.838 54.483))
     (stroke (width 0) (type default))
@@
   )
   (wire (pts (xy 81.915 128.778) (xy 85.217 128.778))
+    (stroke (width 0) (type default))
+  )
+  (wire (pts (xy 204.343 121.158) (xy 204.343 121.031))
     (stroke (width 0) (type default))
   )
@@
     )
   )
-  (symbol (lib_id "Connector_Generic:Conn_01x01") (at 184.531 115.951 90) (unit 1)
-    (in_bom yes) (on_board yes) (dnp no) (fields_autoplaced)
-    (property "Reference" "J7" (at 186.563 114.7389 90)
+  (symbol (lib_id "Connector_Generic:Conn_01x01") (at 204.343 116.078 90) (unit 1)
+    (in_bom yes) (on_board yes) (dnp no) (fields_autoplaced)
+    (property "Reference" "J7" (at 206.375 114.8659 90)
       (effects (font (size 1.27 1.27)) (justify right))
     )
-    (property "Value" "COIL_PWR" (at 186.563 117.1631 90)
+    (property "Value" "COIL_PWR" (at 206.375 117.2901 90)
       (effects (font (size 1.27 1.27)) (justify right))
     )
-    (property "Footprint" "TestPoint:TestPoint_THTPad_2.0x2.0mm_Drill1.0mm" (at 184.531 115.951 0)
-      (effects (font (size 1.27 1.27)) hide)
-    )
-    (property "Datasheet" "~" (at 184.531 115.951 0)
-      (effects (font (size 1.27 1.27)) hide)
-    )
+    (property "Footprint" "TestPoint:TestPoint_THTPad_2.0x2.0mm_Drill1.0mm" (at 204.343 116.078 0)
+      (effects (font (size 1.27 1.27)) hide)
+    )
+    (property "Datasheet" "~" (at 204.343 116.078 0)
+      (effects (font (size 1.27 1.27)) hide)
+    )

Commit message: WIP on PCB
Parts:
- added C14: 220uF, Capacitor_SMD:CP_Elec_6.3x7.7, symbol Device:C_Polarized
- J5: now not fitted
- U7, U8: footprint Package_TO_SOT_SMD:TSOT-23-6 -> Package_TO_SOT_SMD:SOT-23-6_Handsoldering
Connections:
- net GND: now also C14.2
- net at C15.1, L2.1, Q6.2 (D)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: now also C14.1
Changed lines of the file:
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@@
   (junction (at 145.796 53.721) (diameter 0) (color 0 0 0 0)
   )
+  (junction (at 125.73 130.937) (diameter 0) (color 0 0 0 0)
+  )
   (junction (at 170.815 43.815) (diameter 0) (color 0 0 0 0)
   )
@@
     (stroke (width 0) (type default))
   )
+  (wire (pts (xy 125.73 130.937) (xy 140.462 130.937))
+    (stroke (width 0) (type default))
+  )
   (wire (pts (xy 227.838 51.943) (xy 228.473 51.943))
     (stroke (width 0) (type default))
@@
     (stroke (width 0) (type default))
   )
+  (wire (pts (xy 125.73 144.526) (xy 125.73 145.796))
+    (stroke (width 0) (type default))
+  )
   (wire (pts (xy 101.6 40.513) (xy 101.6 43.942))
     (stroke (width 0) (type default))
@@
     (stroke (width 0) (type default))
   )
-  (wire (pts (xy 118.999 130.937) (xy 140.462 130.937))
+  (wire (pts (xy 118.999 130.937) (xy 125.73 130.937))
     (stroke (width 0) (type default))
   )
@@
   )
   (wire (pts (xy 227.838 54.483) (xy 227.838 68.199))
+    (stroke (width 0) (type default))
+  )
+  (wire (pts (xy 125.73 130.937) (xy 125.73 136.906))
     (stroke (width 0) (type default))
   )
@@
     (stroke (width 0) (type default))
     (fill (type none))
-    (effects (font (size 1.27 1.27)) (justify left top))
+    (effects (font (size 1.27 1.27)) (justify right top))
   )
   (text_box "Backlight power supply\n~320mA on output (+24V)\n2A on input (+5V)"
@@
       (effects (font (size 1.27 1.27)))
     )
-    (property "Footprint" "Package_TO_SOT_SMD:TSOT-23-6" (at 158.877 143.637 0)
+    (property "Footprint" "Package_TO_SOT_SMD:SOT-23-6_Handsoldering" (at 158.877 143.637 0)
       (effects (font (size 1.27 1.27)) hide)
     )
@@
       (effects (font (size 1.27 1.27)))
     )
-    (property "Footprint" "Package_TO_SOT_SMD:TSOT-23-6" (at 156.718 66.421 0)
+    (property "Footprint" "Package_TO_SOT_SMD:SOT-23-6_Handsoldering" (at 156.718 66.421 0)
       (effects (font (size 1.27 1.27)) hide)
     )
@@
   )
   (symbol (lib_id "Connector:Conn_01x02_Pin") (at 145.923 31.369 0) (mirror y) (unit 1)
-    (in_bom yes) (on_board yes) (dnp no) (fields_autoplaced)
+    (in_bom yes) (on_board yes) (dnp yes) (fields_autoplaced)
     (property "Reference" "J5" (at 146.6342 31.4269 0)
       (effects (font (size 1.27 1.27)) (justify right))
@@
         )
       )
+    )
+  )
+  (symbol (lib_id "Device:C_Polarized") (at 125.73 140.716 0) (unit 1)
+    (in_bom yes) (on_board yes) (dnp no) (fields_autoplaced)
+    (property "Reference" "C14" (at 128.651 138.6149 0)
+      (effects (font (size 1.27 1.27)) (justify left))
+    )
+    (property "Value" "220uF" (at 128.651 141.0391 0)
+      (effects (font (size 1.27 1.27)) (justify left))
+    )
+    (property "Footprint" "Capacitor_SMD:CP_Elec_6.3x7.7" (at 126.6952 144.526 0)
+      (effects (font (size 1.27 1.27)) hide)
+    )
+    (property "Datasheet" "~" (at 125.73 140.716 0)
+      (effects (font (size 1.27 1.27)) hide)
+    )
+    (property "Voltage" "16V" (at 125.73 140.716 0)
+      (effects (font (size 1.27 1.27)) hide)
+    )
+    (property "LCSC" "C125979" (at 125.73 140.716 0)
+      (effects (font (size 1.27 1.27)) hide)
+    )
+    (pin "1")
+    (pin "2")
+    (instances
+      (project "ESP32-S3_flipdot"
+        (path "/f80df99c-cf65-44b7-a2c8-c57a2edf41e8"
+          (reference "C14") (unit 1)
+        )
+        (path "/f80df99c-cf65-44b7-a2c8-c57a2edf41e8/9fb91dec-c1b1-4168-a997-9a87ad03d4f5"
+          (reference "C12") (unit 1)
+        )
+      )
+    )
+  )
+  (symbol (lib_id "power:GND") (at 125.73 145.796 0) (unit 1)
+    (in_bom yes) (on_board yes) (dnp no) (fields_autoplaced)
+    (property "Reference" "#PWR059" (at 125.73 152.146 0)
+      (effects (font (size 1.27 1.27)) hide)
+    )
+    (property "Value" "GND" (at 125.73 149.9291 0)
+      (effects (font (size 1.27 1.27)))
+    )
+    (property "Footprint" "" (at 125.73 145.796 0)
+      (effects (font (size 1.27 1.27)) hide)
+    )
+    (property "Datasheet" "" (at 125.73 145.796 0)
+      (effects (font (size 1.27 1.27)) hide)
+    )
+    (pin "1")
+    (instances
+      (project "ESP32-S3_flipdot"
+        (path "/f80df99c-cf65-44b7-a2c8-c57a2edf41e8/9fb91dec-c1b1-4168-a997-9a87ad03d4f5"
+          (reference "#PWR059") (unit 1)
+        )
+      )

Commit message: PCB in production!
Parts:
- J3: LCSC C5157144 -> C709041
- J5, J6, J7: now left out of the parts list
- Q3, Q4: footprint Package_TO_SOT_SMD:SOT-23 -> Package_TO_SOT_SMD:SOT-89-3; symbol Transistor_BJT:2N3904 -> Library:2N3904U; LCSC C18536 -> C2928256
Connections:
- net GND: now also Q3.3 (E), Q4.3 (E); no longer Q3.1 (E), Q4.1 (E)
- net at Q5.1 (G), R31.2: now also Q3.2 (C); no longer Q3.3 (C)
- net at Q6.1 (G), R32.2: now also Q4.2 (C); no longer Q4.3 (C)
- net at R28.2, R30.1: now also Q4.1 (B); no longer Q4.2 (B)
- net at R27.2, R29.1: now also Q3.1 (B); no longer Q3.2 (B)
Changed lines of the file:
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@@
   )
   (symbol (lib_id "Connector_Generic:Conn_01x01") (at 202.311 37.465 90) (unit 1)
-    (in_bom yes) (on_board yes) (dnp no) (fields_autoplaced)
+    (in_bom no) (on_board yes) (dnp no) (fields_autoplaced)
     (property "Reference" "J6" (at 204.343 36.2529 90)
       (effects (font (size 1.27 1.27)) (justify right))
@@
   )
   (symbol (lib_id "Connector_Generic:Conn_01x01") (at 204.343 116.078 90) (unit 1)
-    (in_bom yes) (on_board yes) (dnp no) (fields_autoplaced)
+    (in_bom no) (on_board yes) (dnp no) (fields_autoplaced)
     (property "Reference" "J7" (at 206.375 114.8659 90)
       (effects (font (size 1.27 1.27)) (justify right))
@@
       (effects (font (size 1.27 1.27)) hide)
     )
-    (property "LCSC" "C5157144" (at 233.553 51.943 0)
+    (property "LCSC" "C709041" (at 233.553 51.943 0)
       (effects (font (size 1.27 1.27)) hide)
     )
@@
   )
   (symbol (lib_id "Connector:Conn_01x02_Pin") (at 145.923 31.369 0) (mirror y) (unit 1)
-    (in_bom yes) (on_board yes) (dnp yes) (fields_autoplaced)
+    (in_bom no) (on_board yes) (dnp yes) (fields_autoplaced)
     (property "Reference" "J5" (at 146.6342 31.4269 0)
       (effects (font (size 1.27 1.27)) (justify right))
@@
     )
   )
-  (symbol (lib_id "Transistor_BJT:2N3904") (at 99.06 51.562 0) (unit 1)
+  (symbol (lib_id "Library:2N3904U") (at 99.06 51.562 0) (unit 1)
     (in_bom yes) (on_board yes) (dnp no) (fields_autoplaced)
     (property "Reference" "Q3" (at 103.9114 50.3499 0)
@@
       (effects (font (size 1.27 1.27)) (justify left))
     )
-    (property "Footprint" "Package_TO_SOT_SMD:SOT-23" (at 104.14 53.467 0)
+    (property "Footprint" "Package_TO_SOT_SMD:SOT-89-3" (at 104.14 53.467 0)
       (effects (font (size 1.27 1.27) italic) (justify left) hide)
     )
-    (property "Datasheet" "https://www.onsemi.com/pub/Collateral/2N3903-D.PDF" (at 99.06 51.562 0)
+    (property "Datasheet" "https://datasheet.lcsc.com/lcsc/2201121400_CBI-2N3904U_C2928256.pdf" (at 99.06 51.562 0)
       (effects (font (size 1.27 1.27)) (justify left) hide)
     )
-    (property "LCSC" "C18536" (at 99.06 51.562 0)
+    (property "LCSC" "C2928256" (at 99.06 51.562 0)
       (effects (font (size 1.27 1.27)) hide)
     )
@@
     )
   )
-  (symbol (lib_id "Transistor_BJT:2N3904") (at 101.219 128.778 0) (unit 1)
+  (symbol (lib_id "Library:2N3904U") (at 101.219 128.778 0) (unit 1)
     (in_bom yes) (on_board yes) (dnp no) (fields_autoplaced)
     (property "Reference" "Q4" (at 106.0704 127.5659 0)
@@
       (effects (font (size 1.27 1.27)) (justify left))
     )
-    (property "Footprint" "Package_TO_SOT_SMD:SOT-23" (at 106.299 130.683 0)
+    (property "Footprint" "Package_TO_SOT_SMD:SOT-89-3" (at 106.299 130.683 0)
       (effects (font (size 1.27 1.27) italic) (justify left) hide)
     )
-    (property "Datasheet" "https://www.onsemi.com/pub/Collateral/2N3903-D.PDF" (at 101.219 128.778 0)
+    (property "Datasheet" "https://datasheet.lcsc.com/lcsc/2201121400_CBI-2N3904U_C2928256.pdf" (at 101.219 128.778 0)
       (effects (font (size 1.27 1.27)) (justify left) hide)
     )
-    (property "LCSC" "C18536" (at 101.219 128.778 0)
-      (effects (font (size 1.27 1.27)) hide)
-    )
+    (property "LCSC" "C2928256" (at 101.219 128.778 0)
+      (effects (font (size 1.27 1.27)) hide)
+    )
