File: Controller/ESP32-S3_flipdot/ESP32-S3_flipdot.kicad_pcb (KiCad board)
At the start: 2 copper layers, 185 x 75 mm, 91 parts, among them J1 Power in, J2 FTDI, J3 Mobitec display, J4 BackLight, J5 BL_CMD, J6 BL_PWR, J7 COIL_PWR, Q1 BC817, Q2 BC817, Q3 2N3904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

Commit message: Before new dc-dc
Parts:
- added J8: Aux_conn, Connector_PinHeader_2.54mm:PinHeader_1x06_P2.54mm_Vertical, F.Cu at (173.3, 89.4)
- added R37: 0, Resistor_SMD:R_0603_1608Metric, F.Cu at (179.8, 102.2)
- added R38: 0, Resistor_SMD:R_0603_1608Metric, F.Cu at (179.8, 99.0)
- moved TP4 25.8 mm to (138.5, 108.7)
- moved TP2 25.2 mm to (147.9, 108.7)
- moved TP1 19.3 mm to (153.1, 108.7)
- moved TP3 19.2 mm to (143.2, 108.7)
- moved R2 15.1 mm to (170.4, 75.7)
- moved D3 15.1 mm to (170.4, 79.7)
- moved J7 6.68 mm to (68.5, 68.1)
- moved C9 5.32 mm to (112.5, 116.2)
- moved J3 5.32 mm to (115.6, 53.7)
- moved R10 5.32 mm to (111.4, 103.8)
- moved R11 5.32 mm to (82.8, 103.8)
- moved R12 5.32 mm to (88.7, 103.8)
- moved R13 5.32 mm to (97.8, 103.8)
- moved R14 5.32 mm to (108.2, 103.8)
- moved R15 5.32 mm to (113.0, 95.9)
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Connections:
- U2 pad 10: unconnected-(U2-GPIO17/U1TXD/ADC2_CH6-Pad10) -> /ESP32/U1TXD
- U2 pad 11: unconnected-(U2-GPIO18/U1RXD/ADC2_CH7/CLK_OUT3-Pad11) -> /ESP32/U1RXD
- U2 pad 8: unconnected-(U2-GPIO15/U0RTS/ADC2_CH4/XTAL_32K_P-Pad8) -> /ESP32/GPIO15
- U2 pad 9: unconnected-(U2-GPIO16/U0CTS/ADC2_CH5/XTAL_32K_N-Pad9) -> /ESP32/GPIO16
Routing:
- net /ESP32/GPIO15: track 0.00 -> 67.2 mm, vias 0 -> 4
- net /ESP32/U1TXD: track 0.00 -> 66.2 mm, vias 0 -> 6
- net /ESP32/GPIO16: track 0.00 -> 66.1 mm, vias 0 -> 4
- net /ESP32/U1RXD: track 0.00 -> 64.6 mm, vias 0 -> 4
- net +3V3: track 74.4 -> 97.0 mm, vias 0 -> 2
- net GND: track 112.7 -> 90.8 mm, vias 28 -> 86
- net +5V: track 357.8 -> 373.4 mm
- net /Outputs/SER: track 77.7 -> 86.9 mm
- net Vdrive: track 99.5 -> 90.3 mm
- net Net-(J8-Pin_6): track 0.00 -> 8.91 mm
- net /Outputs/SRCLK: track 114.5 -> 121.7 mm
- net /Outputs/~{SRCLR}: track 108.7 -> 115.4 mm
- net /Outputs/RCLK: track 107.4 -> 111.2 mm
- net Net-(U2-GPIO14/TOUCH14/ADC2_CH3/FSPIWP/FSPIDQS/SUBSPIWP): track 11.1 -> 14.7 mm, vias 0 -> 2
Other:
- outline, holes or cut-outs redrawn
- board text added: "+5V"
- board text added: "15"
- board text added: "16"
- board text added: "BOOT"
- board text added: "GND"
- board text added: "LIGHT"
- board text added: "RESET"
- board text added: "RX"
- board text added: "TX"
- board text added: "VCC"
- board text added: "https://github.com/BwanaFr/flipdot-controller"

Commit message: WIP on PCB
Parts:
- added C12: 220uF, Capacitor_SMD:CP_Elec_6.3x7.7, F.Cu at (56.4, 105.4)
- TP1, TP2, TP3, TP4: footprint TestPoint:TestPoint_Pad_1.5x1.5mm -> TestPoint:TestPoint_THTPad_2.0x2.0mm_Drill1.0mm
- U7, U8: footprint Package_TO_SOT_SMD:TSOT-23-6 -> Package_TO_SOT_SMD:SOT-23-6_Handsoldering
- moved J5 35.7 mm to (228.3, 72.0), turned to 180 degrees
- moved Q5 31.5 mm to (226.0, 80.9), turned to -90 degrees
- moved C13 22.0 mm to (226.5, 93.0)
- moved D4 21.5 mm to (202.2, 82.5), turned to 0 degrees
- moved R35 20.0 mm to (53.8, 86.6), turned to -90 degrees
- moved L1 19.1 mm to (214.2, 82.5), turned to 180 degrees
- moved C16 18.9 mm to (201.7, 88.4), turned to -90 degrees
- moved R36 16.5 mm to (56.2, 87.6), turned to 0 degrees
- moved J6 14.1 mm to (200.1, 78.0)
- moved J1 12.6 mm to (216.1, 68.1)
- moved C18 11.8 mm to (192.6, 86.7), turned to -90 degrees
- moved J4 11.4 mm to (216.2, 56.5)
- moved R33 11.0 mm to (207.8, 94.3), turned to 0 degrees
- moved U8 10.9 mm to (57.1, 93.4), turned to -90 degrees
- moved C15 10.7 mm to (55.6, 97.4), turned to 180 degrees
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Connections:
- J1 pad 1: +5V -> GND
- J1 pad 2: GND -> +5V
Routing:
- net +5V: track 373.4 -> 332.1 mm, vias 2 -> 4
- net Net-(D4-K): track 42.9 -> 80.8 mm, vias 0 -> 1
- net GND: track 90.8 -> 128.1 mm, vias 86 -> 125
- net Net-(Q3-C): track 12.3 -> 45.7 mm
- net Net-(Q6-D): track 26.2 -> 0.00 mm
- net /BACKLIGHT_ON: track 100.7 -> 119.4 mm, vias 4 -> 2
- net Net-(D5-A): track 18.5 -> 0.00 mm
- net Vdrive: track 90.3 -> 75.2 mm
- net /Outputs/RCLK: track 111.2 -> 124.8 mm, vias 7 -> 1
- net Net-(D4-A): track 13.4 -> 0.00 mm
- net /Outputs/~{SRCLR}: track 115.4 -> 125.9 mm
- net /ESP32/CHIP_PU: track 92.9 -> 86.4 mm
- net /DC-DC Step-up/+5V_BL: track 12.9 -> 6.73 mm
- net /Outputs/SRCLK: track 121.7 -> 126.6 mm, vias 4 -> 0
- net /Outputs/SER: track 86.9 -> 82.7 mm, vias 4 -> 1
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- added copper zone on F.Cu, net Net-(D4-A)
- added copper zone on F.Cu, net Net-(D5-A)
- added copper zone on F.Cu, net Net-(Q6-D)

Commit message: PCB in production!
Parts:
- Q3, Q4: footprint Package_TO_SOT_SMD:SOT-23 -> Package_TO_SOT_SMD:SOT-89-3
- moved C4 7.66 mm to (145.4, 57.9), turned to -90 degrees
- moved Q3 5.00 mm to (211.7, 112.5), turned to 180 degrees
- moved R1 4.07 mm to (143.1, 57.2), turned to 0 degrees
- moved R29 3.25 mm to (217.7, 114.0)
- moved R27 1.50 mm to (217.7, 118.1)
- moved Q4 1.27 mm to (63.6, 116.6), turned to 180 degrees
Connections:
- Q3 pad 1: GND -> Net-(Q3-B)
- Q3 pad 2: Net-(Q3-B) -> Net-(Q3-C)
- Q3 pad 3: Net-(Q3-C) -> GND
- Q4 pad 1: GND -> Net-(Q4-B)
- Q4 pad 2: Net-(Q4-B) -> Net-(Q4-C)
- Q4 pad 3: Net-(Q4-C) -> GND
Routing:
- net /ESP32/DTR: track 14.1 -> 25.6 mm, vias 2 -> 0
- net /ESP32/CHIP_PU: track 86.4 -> 79.7 mm
- net Net-(Q3-C): track 45.7 -> 49.1 mm
- net +5V: track 332.1 -> 329.7 mm
- net /BACKLIGHT_ON: track 119.4 -> 117.4 mm
- net Net-(Q3-B): track 4.92 -> 6.86 mm
- net Net-(Q4-C): track 8.39 -> 10.1 mm
- net /ESP32/GPIO0: track 37.0 -> 38.5 mm
- net Net-(D2-A): track 11.3 -> 9.77 mm
- net GND: track 128.1 -> 126.7 mm, vias 125 -> 141
- net /ESP32/U0TXD: track 16.9 -> 16.3 mm, vias 4 -> 2
- net /ESP32/U0RXD: vias 4 -> 2
- net (no net): vias 10 -> 0
Other:
- outline, holes or cut-outs redrawn
