File: Controller/ESP32-S3_flipdot/esp32.kicad_sch (KiCad schematic)
At the start: 23 parts, among them J2 FTDI, Q1 BC817, Q2 BC817, SW1 Reset, SW2 Boot, U1 LM1117MP-3.3, U2 ESP32-S3-WROOM-1U-N16R8

Commit message: Before new dc-dc
Parts:
- added J8: Aux_conn, Connector_PinHeader_2.54mm:PinHeader_1x06_P2.54mm_Vertical, symbol Connector_Generic:Conn_01x06
- added R37, R38: 0, Resistor_SMD:R_0603_1608Metric, symbol Device:R
Connections:
- net +3V3: now also R38.1
- net +5V: now also R37.1
- net GND: now also J8.1 (Pin_1)
- net U1TXD: now reaches U2.10 (GPIO17/U1TXD/ADC2_CH6)
- net U1TXD: now also J8.5 (Pin_5)
- net U1RXD: now reaches U2.11 (GPIO18/U1RXD/ADC2_CH7/CLK_OUT3)
- net U1RXD: now also J8.4 (Pin_4)
- net GPIO15: now reaches U2.8 (GPIO15/U0RTS/ADC2_CH4/XTAL_32K_P)
- net GPIO15: now also J8.2 (Pin_2)
- net GPIO16: now reaches U2.9 (GPIO16/U0CTS/ADC2_CH5/XTAL_32K_N)
- net GPIO16: now also J8.3 (Pin_3)
- new net: J8.6 (Pin_6), R37.2, R38.2
Other:
- moved on the sheet: D3, R2

Commit message: PCB in production!
Parts:
- J8, R37, R38: now left out of the parts list
Changed lines of the file:
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@@
   )
   (symbol (lib_id "Device:R") (at 76.073 77.724 0) (unit 1)
-    (in_bom yes) (on_board yes) (dnp yes) (fields_autoplaced)
+    (in_bom no) (on_board yes) (dnp yes) (fields_autoplaced)
     (property "Reference" "R38" (at 77.851 76.5119 0)
       (effects (font (size 1.27 1.27)) (justify left))
@@
   )
   (symbol (lib_id "Connector_Generic:Conn_01x06") (at 50.546 92.329 180) (unit 1)
-    (in_bom yes) (on_board yes) (dnp yes) (fields_autoplaced)
+    (in_bom no) (on_board yes) (dnp yes) (fields_autoplaced)
     (property "Reference" "J8" (at 50.546 79.2947 0)
       (effects (font (size 1.27 1.27)))
@@
   )
   (symbol (lib_id "Device:R") (at 64.135 77.597 0) (unit 1)
-    (in_bom yes) (on_board yes) (dnp yes) (fields_autoplaced)
+    (in_bom no) (on_board yes) (dnp yes) (fields_autoplaced)
     (property "Reference" "R37" (at 65.913 76.3849 0)
       (effects (font (size 1.27 1.27)) (justify left))

Commit message: Progress on controller firmware
Parts:
- SW1, SW2: LCSC C512395 -> C528967
Changed lines of the file:
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@@
       (effects (font (size 1.27 1.27)) hide)
     )
-    (property "LCSC" "C512395" (at 92.075 180.975 0)
+    (property "LCSC" "C528967" (at 92.075 180.975 0)
       (effects (font (size 1.27 1.27)) hide)
     )
@@
       (effects (font (size 1.27 1.27)) hide)
     )
-    (property "LCSC" "C512395" (at 76.835 181.61 90)
-      (effects (font (size 1.27 1.27)) hide)
-    )
+    (property "LCSC" "C528967" (at 76.835 181.61 90)
+      (effects (font (size 1.27 1.27)) hide)
+    )
